Commit message: modify arena, disable gripper

File: mir_common/mir_description/urdf/sensor_mounts/intel_f200_camera_mount.urdf.xacro (robot description, xacro)
@@ -17,5 +17,5 @@
 			</inertial>
 			<visual>
-				<origin xyz="0 0 0" rpy="-${M_PI/2} 0 -${M_PI/2}" />
+				<origin xyz="0 0 -0.01" rpy="-${M_PI/2} 0 -${M_PI/2}" />
 				<geometry>
 					<mesh filename="package://mir_description/meshes/sensor_mounts/intel_f200_camera_mount.dae" scale="0.001 0.001 0.001" />

File: mir_robots/mir_hardware_config/youbot-brsu-1/urdf/robot.urdf.xacro (robot description, xacro)
@@ -15,5 +15,5 @@
   <xacro:include filename="$(find youbot_description)/urdf/youbot_arm/arm.urdf.xacro"/>
   <xacro:include filename="$(find mir_description)/urdf/misc/adapter_plate.urdf.xacro" />
-  <xacro:include filename="$(find mir_description)/urdf/grippers/dynamixel/v1/dynamixel_gripper.urdf.xacro" />
+  <!--xacro:include filename="$(find mir_description)/urdf/grippers/dynamixel/v1/dynamixel_gripper.urdf.xacro" /-->
   <!-- controller manager -->
   <xacro:include filename="$(find youbot_description)/controller/ros_controller.urdf.xacro" />
@@ -49,6 +49,6 @@
     <origin xyz="-0.075 0.024 0.04" rpy="0 ${-M_PI / 2} 0" />
   </xacro:intel_realsense_f200_camera>
-  <xacro:dynamixel_gripper name="gripper" parent="arm_link_5">
+  <!--xacro:dynamixel_gripper name="gripper" parent="arm_link_5">
     <origin xyz="0 0 -0.02" rpy="0 0 0" />
-  </xacro:dynamixel_gripper>
+  </xacro:dynamixel_gripper-->
 </robot>

File: mir_robots/mir_hardware_config/youbot-brsu-2/urdf/robot.urdf.xacro (robot description, xacro)
@@ -24,4 +24,6 @@
   <xacro:include filename="$(find mir_description)/urdf/sensor_mounts/intel_f200_camera_mount.urdf.xacro"/>
   <xacro:include filename="$(find mcr_description)/urdf/sensors/intel_realsense_f200_camera.urdf.xacro"/>
+  <!--Stereo camera-->
+  <!--xacro:include filename="$(find flying_gazebo_stereo_cam)/model/flying_stereo_cam.xacro" /-->
   <!-- Now we can start using the macros included above to define the actual youbot -->
   <!-- standard youBot configuration -->
@@ -46,14 +48,21 @@
      <origin xyz="-0.3 0.0 -0.035" rpy="${M_PI} 0 ${M_PI}" />
   </xacro:hokuyo_urg04_laser>
-  <xacro:dynamixel_gripper_v2 name="gripper" parent="arm_link_5">
-    <origin xyz="0.003 0 0.0052" rpy="0 0 0" />
-  </xacro:dynamixel_gripper_v2>
+  <!--xacro:dynamixel_gripper_v2 name="gripper" parent="arm_link_5">
+    <origin xyz="0.0 0 0.0" rpy="0 0 0" />
+  </xacro:dynamixel_gripper_v2-->
   <!-- camera mount for Intel RealSense F200 -->
-  <xacro:intel_f200_camera_mount name="camera_mount" parent="gripper_motor_mount_link">
+  <!--xacro:intel_f200_camera_mount name="camera_mount" parent="gripper_motor_mount_link">
+    <origin xyz="-0.00375 -0.0007 0.012" rpy="0.06 -0.04 0" />
+  </xacro:intel_f200_camera_mount-->
+  <xacro:intel_f200_camera_mount name="camera_mount" parent="arm_link_5">
     <origin xyz="-0.00375 -0.0007 0.012" rpy="0.06 -0.04 0" />
   </xacro:intel_f200_camera_mount>
   <!-- 3D camera on arm -->
   <xacro:intel_realsense_f200_camera name="arm_cam3d" parent="camera_mount_link">
+    <origin xyz="-0.0415 -0.00 0.018" rpy="0.0 -${M_PI/2} 0.0" />
+  </xacro:intel_realsense_f200_camera>
+  <!--Stereo camera-->
+   <!--xacro:flying_stereo_cam name="camera" parent="camera_mount_link">
     <origin xyz="-0.045 -0.00 0.00" rpy="0.0 -${M_PI/2} 0.0" />
-  </xacro:intel_realsense_f200_camera>
+  </xacro:flying_stereo_cam-->
 </robot>

File: mir_robots/mir_hardware_config/youbot-brsu-3/urdf/robot.urdf.xacro (robot description, xacro)
@@ -15,5 +15,5 @@
   <xacro:include filename="$(find youbot_description)/urdf/youbot_arm/arm.urdf.xacro"/>
   <xacro:include filename="$(find mir_description)/urdf/misc/adapter_plate.urdf.xacro" />
-  <xacro:include filename="$(find mir_description)/urdf/grippers/dynamixel/v2/dynamixel_gripper.urdf.xacro" />
+  <!--xacro:include filename="$(find mir_description)/urdf/grippers/dynamixel/v2/dynamixel_gripper.urdf.xacro" /-->
   <!-- controller manager -->
   <xacro:include filename="$(find youbot_description)/controller/ros_controller.urdf.xacro" />
@@ -46,7 +46,7 @@
      <origin xyz="-0.3 0.0 -0.035" rpy="0 0 ${M_PI}" />
   </xacro:hokuyo_urg04_laser>
-  <xacro:dynamixel_gripper_v2 name="gripper" parent="arm_link_5">
+  <!--xacro:dynamixel_gripper_v2 name="gripper" parent="arm_link_5">
     <origin xyz="0.003 0 0.0052" rpy="0 0 0" />
-  </xacro:dynamixel_gripper_v2>
+  </xacro:dynamixel_gripper_v2-->
   <!-- camera mount for Intel RealSense F200 -->
   <xacro:intel_f200_camera_mount name="camera_mount" parent="gripper_motor_mount_link">

File: mir_robots/mir_hardware_config/youbot-brsu-4/urdf/robot.urdf.xacro (robot description, xacro)
@@ -15,5 +15,5 @@
   <xacro:include filename="$(find youbot_description)/urdf/youbot_arm/arm.urdf.xacro"/>
   <xacro:include filename="$(find mir_description)/urdf/misc/adapter_plate.urdf.xacro" />
-  <xacro:include filename="$(find mir_description)/urdf/grippers/dynamixel/v2/dynamixel_gripper.urdf.xacro" />
+  <!--xacro:include filename="$(find mir_description)/urdf/grippers/dynamixel/v2/dynamixel_gripper.urdf.xacro" /-->
   <!-- controller manager -->
   <xacro:include filename="$(find youbot_description)/controller/ros_controller.urdf.xacro" />
@@ -46,7 +46,7 @@
      <origin xyz="-0.3 0.0 -0.035" rpy="${M_PI} 0 ${M_PI}" />
   </xacro:hokuyo_urg04_laser>
-  <xacro:dynamixel_gripper_v2 name="gripper" parent="arm_link_5">
+  <!--xacro:dynamixel_gripper_v2 name="gripper" parent="arm_link_5">
     <origin xyz="0.003 0 0.0052" rpy="0 0 0" />
-  </xacro:dynamixel_gripper_v2>
+  </xacro:dynamixel_gripper_v2-->
   <!-- camera mount for Intel RealSense F200 -->
   <xacro:intel_f200_camera_mount name="camera_mount" parent="gripper_motor_mount_link">
